Commit message: Refinement

File: urdf/arm4dof.urdf (robot description, URDF)
Before this commit: robot arm4dof, 6 links, 5 joints
Links:
- removed link hand_fixed
- removed link hand_free
- added link finger, mass 0.1620904614417843; collision mesh filename=package://arm4dof_description/meshes/finger.stl scale=1.0 1.0 1.0; visual mesh filename=package://arm4dof_description/meshes/finger.stl scale=1.0 1.0 1.0
- added link hand, mass 0.751568194075787; collision mesh filename=package://arm4dof_description/meshes/hand.stl scale=1.0 1.0 1.0; visual mesh filename=package://arm4dof_description/meshes/hand.stl scale=1.0 1.0 1.0
Joints:
- removed joint rev0
- removed joint rev1
- removed joint rev2
- removed joint rev3
- removed joint rev4
- added joint finger_joint: type revolute, parent hand, child finger, origin xyz=-0.017899999999822058 0.038515074085115855 0.06678500064820125 rpy=0 0 0, axis -1.0000000000000007 -5.5511151231176124e-17 -7.216449660063521e-16, limit lower=-0.785 upper=0.785 effort=0 velocity=0
- added joint joint1: type revolute, parent forearm, child hand, origin xyz=-1.9312351197398048e-17 4.388850394221322e-16 0.09999999999999948 rpy=0 0 0, axis 5.469212746514901e-15 -0.9999999999999988 4.0132109545040804e-15, limit lower=-2.355 upper=2.355 effort=0 velocity=0
- added joint joint2: type revolute, parent upperarm, child forearm, origin xyz=-1.7781568860571195e-13 -7.408511604189982e-08 0.09157000000000029 rpy=0 0 0, axis -4.56250541873071e-15 -0.9999999999999984 4.013210954504077e-15, limit lower=-2.355 upper=2.355 effort=0 velocity=0
- added joint joint3: type revolute, parent shoulder, child upperarm, origin xyz=2.7934012189739094e-08 -0.01790000000000031 0.030099999351800136 rpy=0 0 0, axis 4.9960036108131995e-16 -0.9999999999999996 1.1662307446965333e-14, limit lower=-2.355 upper=2.355 effort=0 velocity=0
- added joint joint4: type revolute, parent base_link, child shoulder, origin xyz=-0.00011998774492904957 0.009207659539338426 0.009127545265139512 rpy=0 0 0, axis 1.1102230246251564e-16 -2.7660707925536432e-17 0.9999999999999997, limit lower=-3.14 upper=3.14 effort=0 velocity=0

Commit message: 実機に合わせてURDF作り直し

File: urdf/arm4dof.urdf (robot description, URDF)
Before this commit: robot arm4dof, 6 links, 5 joints
Links:
- added link fixfinger; visual box size=0.025 0.005 0.09
- link base_link: mass 0.7502954240514383 -> None; geometry visual cylinder length=0.04 radius=0.05
- link finger: mass 0.1620904614417843 -> None; geometry visual box size=0.025 0.005 0.09
- link forearm: mass 0.13426852980149212 -> None; geometry visual box size=0.02473 0.036 0.124
- link hand: mass 0.751568194075787 -> None; geometry visual box size=0.02473 0.0549 0.089265
- link shoulder: mass 0.07247169619111539 -> None; geometry visual cylinder length=0.006 radius=0.01
- link upperarm: mass 0.6184540010783673 -> None; geometry visual box size=0.02473 0.036 0.11180
Joints:
- added joint fixfinger_joint: type fixed, parent hand, child fixfinger, origin xyz=0 0.036492 0.066785 rpy=0 0 0
- joint finger_joint: axis -1.0000000000000007 -5.5511151231176124e-17 -7.216449660063521e-16 -> (none); origin xyz=-0.017899999999822058 0.038515074085115855 0.06678500064820125 rpy=0 0 0 -> xyz=0 -0.020615 0.066785 rpy=0 0 3.14
- joint joint1: axis 5.469212746514901e-15 -0.9999999999999988 4.0132109545040804e-15 -> 0 0 1; child hand -> shoulder; limit lower=-2.355 upper=2.355 effort=0 velocity=0 -> lower=-3.14 upper=3.14 effort=0 velocity=0; origin xyz=-1.9312351197398048e-17 4.388850394221322e-16 0.09999999999999948 rpy=0 0 0 -> xyz=0 0 0.040 rpy=3.14 0 0; parent forearm -> base_link
- joint joint2: axis -4.56250541873071e-15 -0.9999999999999984 4.013210954504077e-15 -> 0 1 0; child forearm -> upperarm; limit lower=-2.355 upper=2.355 effort=0 velocity=0 -> lower=-1.5708 upper=1.5708 effort=0 velocity=0; origin xyz=-1.7781568860571195e-13 -7.408511604189982e-08 0.09157000000000029 rpy=0 0 0 -> xyz=0 0 -0.029 rpy=3.14 0 0; parent upperarm -> shoulder
- joint joint3: axis 4.9960036108131995e-16 -0.9999999999999996 1.1662307446965333e-14 -> 0 1 0; child upperarm -> forearm; limit lower=-2.355 upper=2.355 effort=0 velocity=0 -> lower=-1.5708 upper=1.5708 effort=0 velocity=0; origin xyz=2.7934012189739094e-08 -0.01790000000000031 0.030099999351800136 rpy=0 0 0 -> xyz=0 0 0.09157 rpy=0 0 0; parent shoulder -> upperarm
- joint joint4: axis 1.1102230246251564e-16 -2.7660707925536432e-17 0.9999999999999997 -> 0 1 0; child shoulder -> hand; limit lower=-3.14 upper=3.14 effort=0 velocity=0 -> lower=-1.5708 upper=1.5708 effort=0 velocity=0; origin xyz=-0.00011998774492904957 0.009207659539338426 0.009127545265139512 rpy=0 0 0 -> xyz=0 0 0.10 rpy=0 0 0; parent base_link -> forearm

Commit message: Update arm4dof.urdf

File: urdf/arm4dof.urdf (robot description, URDF)
Before this commit: robot arm4dof, 7 links, 6 joints
Links:
- link base_link: geometry collision cylinder length=0.04 radius=0.05; visual cylinder length=0.04 radius=0.05
- link finger: geometry collision box size=0.025 0.005 0.09; visual box size=0.025 0.005 0.09
- link fixfinger: geometry collision box size=0.025 0.005 0.09; visual box size=0.025 0.005 0.09
- link forearm: geometry collision box size=0.02473 0.036 0.124; visual box size=0.02473 0.036 0.124
- link hand: geometry collision box size=0.02473 0.0549 0.089265; visual box size=0.02473 0.0549 0.089265
- link shoulder: geometry collision cylinder length=0.006 radius=0.01; visual cylinder length=0.006 radius=0.01
- link upperarm: geometry collision box size=0.02473 0.036 0.11180; visual box size=0.02473 0.036 0.11180
Joints:
- joint joint1: origin xyz=0 0 0.040 rpy=3.14 0 0 -> xyz=0 0 0.040 rpy=0 0 0
- joint joint2: origin xyz=0 0 -0.029 rpy=3.14 0 0 -> xyz=0 0 0.029 rpy=0 0 0
